Commit message: add Isaac Sim ROS2 action graph for autolife

File: src/autolife_description/urdf/autolife.urdf (robot description, URDF)
Before this commit: robot autolife, 47 links, 46 joints
Links:
- link Link_Ankle_to_Knee: geometry collision mesh filename=../meshes/autolife/Link_Ankle_to_Knee.STL; visual mesh filename=../meshes/autolife/Link_Ankle_to_Knee.STL
- link Link_Camera_Gripper_Left: geometry collision mesh filename=../meshes/autolife/Link_Camera_Gripper_Left.STL; visual mesh filename=../meshes/autolife/Link_Camera_Gripper_Left.STL
- link Link_Camera_Gripper_Right: geometry collision mesh filename=../meshes/autolife/Link_Camera_Gripper_Right.STL; visual mesh filename=../meshes/autolife/Link_Camera_Gripper_Right.STL
- link Link_Camera_Head_Back: geometry collision mesh filename=../meshes/autolife/Link_Camera_Head_Back.STL; visual mesh filename=../meshes/autolife/Link_Camera_Head_Back.STL
- link Link_Camera_Head_Forehead: geometry collision mesh filename=../meshes/autolife/Link_Camera_Head_Forehead.STL; visual mesh filename=../meshes/autolife/Link_Camera_Head_Forehead.STL
- link Link_Camera_Head_Left_Eye: geometry collision mesh filename=../meshes/autolife/Link_Camera_Head_Left_Eye.STL; visual mesh filename=../meshes/autolife/Link_Camera_Head_Left_Eye.STL
- link Link_Camera_Head_Right_Eye: geometry collision mesh filename=../meshes/autolife/Link_Camera_Head_Right_Eye.STL; visual mesh filename=../meshes/autolife/Link_Camera_Head_Right_Eye.STL
- link Link_Ground_Vehicle: geometry collision mesh filename=../meshes/autolife/Link_Ground_Vehicle.STL; visual mesh filename=../meshes/autolife/Link_Ground_Vehicle.STL
- link Link_IMU: geometry collision mesh filename=../meshes/autolife/Link_IMU.STL; visual mesh filename=../meshes/autolife/Link_IMU.STL
- link Link_Knee_to_Waist_Pitch: geometry collision mesh filename=../meshes/autolife/Link_Knee_to_Waist_Pitch.STL; visual mesh filename=../meshes/autolife/Link_Knee_to_Waist_Pitch.STL
- link Link_Left_Elbow_to_Forearm: geometry collision mesh filename=../meshes/autolife/Link_Left_Elbow_to_Forearm.STL; visual mesh filename=../meshes/autolife/Link_Left_Elbow_to_Forearm.STL
- link Link_Left_Forearm_to_Wrist_Upper: geometry collision mesh filename=../meshes/autolife/Link_Left_Forearm_to_Wrist_Upper.STL; visual mesh filename=../meshes/autolife/Link_Left_Forearm_to_Wrist_Upper.STL
- link Link_Left_Gripper: geometry collision mesh filename=../meshes/autolife/Link_Left_Gripper.STL; visual mesh filename=../meshes/autolife/Link_Left_Gripper.STL
- link Link_Left_Gripper_Left_Finger: geometry collision mesh filename=../meshes/autolife/Link_Left_Gripper_Left_Finger.STL; visual mesh filename=../meshes/autolife/Link_Left_Gripper_Left_Finger.STL
- link Link_Left_Gripper_Left_Inner_Knuckle: geometry collision mesh filename=../meshes/autolife/Link_Left_Gripper_Left_Inner_Knuckle.STL; visual mesh filename=../meshes/autolife/Link_Left_Gripper_Left_Inner_Knuckle.STL
- link Link_Left_Gripper_Right_Finger: geometry collision mesh filename=../meshes/autolife/Link_Left_Gripper_Right_Finger.STL; visual mesh filename=../meshes/autolife/Link_Left_Gripper_Right_Finger.STL
- link Link_Left_Gripper_Right_Inner_Knuckle: geometry collision mesh filename=../meshes/autolife/Link_Left_Gripper_Right_Inner_Knuckle.STL; visual mesh filename=../meshes/autolife/Link_Left_Gripper_Right_Inner_Knuckle.STL
- link Link_Left_Gripper_Right_Outer_Knuckle: geometry collision mesh filename=../meshes/autolife/Link_Left_Gripper_Right_Outer_Knuckle.STL; visual mesh filename=../meshes/autolife/Link_Left_Gripper_Right_Outer_Knuckle.STL
- link Link_Left_Shoulder_Inner_to_Shoulder_Outer: geometry collision mesh filename=../meshes/autolife/Link_Left_Shoulder_Inner_to_Shoulder_Out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; visual mesh filename=../meshes/autolife/Link_Left_Shoulder_Inner_to_Shoulder_Out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
- link Link_Left_Shoulder_Outer_to_UpperArm: geometry collision mesh filename=../meshes/autolife/Link_Left_Shoulder_Outer_to_UpperArm.STL; visual mesh filename=../meshes/autolife/Link_Left_Shoulder_Outer_to_UpperArm.STL
- link Link_Left_UpperArm_to_Elbow: geometry collision mesh filename=../meshes/autolife/Link_Left_UpperArm_to_Elbow.STL; visual mesh filename=../meshes/autolife/Link_Left_UpperArm_to_Elbow.STL
- link Link_Left_Wrist_Lower_to_Gripper: geometry collision mesh filename=../meshes/autolife/Link_Left_Wrist_Lower_to_Gripper.STL; visual mesh filename=../meshes/autolife/Link_Left_Wrist_Lower_to_Gripper.STL
- link Link_Left_Wrist_Upper_to_Wrist_Lower: geometry collision mesh filename=../meshes/autolife/Link_Left_Wrist_Upper_to_Wrist_Lower.STL; visual mesh filename=../meshes/autolife/Link_Left_Wrist_Upper_to_Wrist_Lower.STL
- link Link_Lidar_Back: geometry collision mesh filename=../meshes/autolife/Link_Lidar_Back.STL; visual mesh filename=../meshes/autolife/Link_Lidar_Back.STL
- link Link_Lidar_Front: geometry collision mesh filename=../meshes/autolife/Link_Lidar_Front.STL; visual mesh filename=../meshes/autolife/Link_Lidar_Front.STL
- link Link_Neck_Pitch_to_Neck_Yaw: geometry collision mesh filename=../meshes/autolife/Link_Neck_Pitch_to_Neck_Yaw.STL; visual mesh filename=../meshes/autolife/Link_Neck_Pitch_to_Neck_Yaw.STL
- link Link_Neck_Roll_to_Neck_Pitch: geometry collision mesh filename=../meshes/autolife/Link_Neck_Roll_to_Neck_Pitch.STL; visual mesh filename=../meshes/autolife/Link_Neck_Roll_to_Neck_Pitch.STL
- link Link_Neck_Yaw_to_Head: geometry collision mesh filename=../meshes/autolife/Link_Neck_Yaw_to_Head.STL; visual mesh filename=../meshes/autolife/Link_Neck_Yaw_to_Head.STL
- link Link_Right_Elbow_to_Forearm: geometry collision mesh filename=../meshes/autolife/Link_Right_Elbow_to_Forearm.STL; visual mesh filename=../meshes/autolife/Link_Right_Elbow_to_Forearm.STL
- link Link_Right_Forearm_to_Wrist_Upper: geometry collision mesh filename=../meshes/autolife/Link_Right_Forearm_to_Wrist_Upper.STL; visual mesh filename=../meshes/autolife/Link_Right_Forearm_to_Wrist_Upper.STL
- link Link_Right_Gripper: geometry collision mesh filename=../meshes/autolife/Link_Right_Gripper.STL; visual mesh filename=../meshes/autolife/Link_Right_Gripper.STL
- link Link_Right_Gripper_Left_Finger: geometry collision mesh filename=../meshes/autolife/Link_Right_Gripper_Left_Finger.STL; visual mesh filename=../meshes/autolife/Link_Right_Gripper_Left_Finger.STL
- link Link_Right_Gripper_Left_Inner_Knuckle: geometry collision mesh filename=../meshes/autolife/Link_Right_Gripper_Left_Inner_Knuckle.STL; visual mesh filename=../meshes/autolife/Link_Right_Gripper_Left_Inner_Knuckle.STL
- link Link_Right_Gripper_Right_Finger: geometry collision mesh filename=../meshes/autolife/Link_Right_Gripper_Right_Finger.STL; visual mesh filename=../meshes/autolife/Link_Right_Gripper_Right_Finger.STL
- link Link_Right_Gripper_Right_Inner_Knuckle: geometry collision mesh filename=../meshes/autolife/Link_Right_Gripper_Right_Inner_Knuckle.S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; visual mesh filename=../meshes/autolife/Link_Right_Gripper_Right_Inner_Knuckle.S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
- link Link_Right_Gripper_Right_Outer_Knuckle: geometry collision mesh filename=../meshes/autolife/Link_Right_Gripper_Right_Outer_Knuckle.S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; visual mesh filename=../meshes/autolife/Link_Right_Gripper_Right_Outer_Knuckle.S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
- link Link_Right_Shoulder_Inner_to_Shoulder_Outer: geometry collision mesh filename=../meshes/autolife/Link_Right_Shoulder_Inner_to_Shoulder_Ou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; visual mesh filename=../meshes/autolife/Link_Right_Shoulder_Inner_to_Shoulder_Ou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
- link Link_Right_Shoulder_Outer_to_UpperArm: geometry collision mesh filename=../meshes/autolife/Link_Right_Shoulder_Outer_to_UpperArm.STL; visual mesh filename=../meshes/autolife/Link_Right_Shoulder_Outer_to_UpperArm.STL
- link Link_Right_UpperArm_to_Elbow: geometry collision mesh filename=../meshes/autolife/Link_Right_UpperArm_to_Elbow.STL; visual mesh filename=../meshes/autolife/Link_Right_UpperArm_to_Elbow.STL
- link Link_Right_Wrist_Lower_to_Gripper: geometry collision mesh filename=../meshes/autolife/Link_Right_Wrist_Lower_to_Gripper.STL; visual mesh filename=../meshes/autolife/Link_Right_Wrist_Lower_to_Gripper.STL
- link Link_Right_Wrist_Upper_to_Wrist_Lower: geometry collision mesh filename=../meshes/autolife/Link_Right_Wrist_Upper_to_Wrist_Lower.STL; visual mesh filename=../meshes/autolife/Link_Right_Wrist_Upper_to_Wrist_Lower.STL
- link Link_Waist_Pitch_to_Waist_Yaw: geometry collision mesh filename=../meshes/autolife/Link_Waist_Pitch_to_Waist_Yaw.STL; visual mesh filename=../meshes/autolife/Link_Waist_Pitch_to_Waist_Yaw.STL
- link Link_Waist_Yaw_to_Shoulder_Inner: geometry collision mesh filename=../meshes/autolife/Link_Waist_Yaw_to_Shoulder_Inner.STL; visual mesh filename=../meshes/autolife/Link_Waist_Yaw_to_Shoulder_Inner.STL
